File: E-throttle/E-throttle.kicad_pcb (KiCad board)
At the start: 2 copper layers, 100 x 100 mm, 68 parts, among them IC1 BTS441TG, J1 Conn_01x15_Socket, J2 Conn_01x15_Socket, J3 Conn_01x11, J4 Conn_01x11, J5 776087-1, J9 Micro_SD_Card, Q1 NMOS, SW1 SW_Push, U1 74HC123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

Commit message: Fixed clearance issues to comply with DRC
Routing:
- net +3V3: track 328.6 -> 310.8 mm
- net /APPS-SIG2-OUT: track 11.5 -> 22.0 mm
- net unconnected-(U5-GND-Pad17): track 2.04 -> 0.54 mm, vias 1 -> 0
- net /SPI-SCK: vias 6 -> 7
Changed lines of the file:
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@@
 		(embedded_fonts no)
 	)
-	(gr_line
-		(start 181.72 103.82)
-		(end 174.72 111.32)
-		(stroke
-			(width 0.2)
-			(type default)
-		)
-		(layer "F.Cu")
-		(net 51)
-	)
 	(gr_arc
 		(start 154.72 38.59)
@@
 	)
 	(segment
-		(start 214.59246 117.157459)
-		(end 214.59246 116.601786)
-		(width 0.5)
-		(layer "F.Cu")
-		(net 5)
-	)
-	(segment
 		(start 225.795001 128.36)
 		(end 226.77 128.36)
@@
 	)
 	(segment
-		(start 225.795001 128.36)
-		(end 214.59246 117.157459)
-		(width 0.5)
-		(layer "F.Cu")
-		(net 5)
-	)
-	(segment
 		(start 163.18 60.36)
 		(end 163.18 57.82)
@@
 	)
 	(segment
-		(start 213.882487 115.891813)
-		(end 212.502433 115.891813)
-		(width 0.5)
-		(layer "F.Cu")
-		(net 5)
-	)
-	(segment
 		(start 211.42 73.62)
 		(end 205.22 79.82)
@@
 	)
 	(segment
+		(start 176.4575 93.0825)
+		(end 176.4575 93.82)
+		(width 0.25)
+		(layer "F.Cu")
+		(net 15)
+	)
+	(segment
 		(start 202.72 104.519813)
 		(end 213.19246 104.519813)
@@
 	)
 	(segment
-		(start 178.808187 90.731813)
-		(end 176.4575 93.0825)
+		(start 178.72 90.82)
+		(end 183.72 90.82)
 		(width 0.25)
 		(layer "F.Cu")
@@
 	)
 	(segment
-		(start 176.4575 93.0825)
-		(end 176.4575 93.82)
+		(start 178.22 91.32)
+		(end 176.4575 93.0825)
 		(width 0.25)
 		(layer "F.Cu")
@@
 	)
 	(segment
-		(start 189.72 90.731813)
-		(end 178.808187 90.731813)
+		(start 178.72 90.82)
+		(end 178.22 91.32)
 		(width 0.25)
 		(layer "F.Cu")
@@
 	)
 	(via
-		(at 189.72 90.731813)
+		(at 183.72 90.82)
 		(size 0.6)
 		(drill 0.3)
@@
 	)
 	(via
+		(at 183.72 90.82)
+		(size 0.6)
+		(drill 0.3)
+		(layers "F.Cu" "B.Cu")
+		(net 15)
+	)
+	(via
 		(at 234.22 95.32)
 		(size 0.6)
@@
 	)
 	(segment
-		(start 189.72 90.731813)
+		(start 190.72 91.731813)
+		(end 190.72 96.705298)
+		(width 0.25)
+		(layer "B.Cu")
+		(net 15)
+	)
+	(segment
+		(start 189.632 90.643813)
 		(end 190.72 91.731813)
 		(width 0.25)
@@
 	)
 	(segment
-		(start 190.72 91.731813)
-		(end 190.72 96.705298)
+		(start 198.534515 104.519813)
+		(end 202.72 104.519813)
 		(width 0.25)
 		(layer "B.Cu")
@@
 	)
 	(segment
+		(start 183.896187 90.643813)
+		(end 189.632 90.643813)
+		(width 0.25)
+		(layer "B.Cu")
+		(net 15)
+	)
+	(segment
 		(start 174.22 95.82)
 		(end 175.72 95.82)
@@
 	)
 	(segment
-		(start 198.534515 104.519813)
-		(end 202.72 104.519813)
+		(start 183.72 90.82)
+		(end 183.896187 90.643813)
 		(width 0.25)
 		(layer "B.Cu")
@@
 	)
 	(segment
+		(start 176.545 98.32)
+		(end 176.545 97.995)
+		(width 0.25)
+		(layer "F.Cu")
+		(net 17)
+	)
+	(segment
 		(start 175.5585 99.3065)
 		(end 175.5585 102.515514)
@@
 	)
 	(segment
+		(start 188.279576 93.183813)
+		(end 188.367576 93.271813)
+		(width 0.25)
+		(layer "F.Cu")
+		(net 17)
+	)
+	(segment
 		(start 176.545 98.32)
 		(end 175.5585 99.3065)
@@
 	)
 	(segment
-		(start 176.545 98.32)
-		(end 176.545 97.995)
+		(start 175.5585 102.515514)
+		(end 175.228014 102.846)
 		(width 0.25)
 		(layer "F.Cu")
@@
 	)
 	(segment
-		(start 176.545 97.995)
-		(end 181.268187 93.271813)
+		(start 187.305344 93.183813)
+		(end 188.279576 93.183813)
 		(width 0.25)
 		(layer "F.Cu")
@@
 	)
 	(segment
-		(start 175.5585 102.515514)
-		(end 175.228014 102.846)
+		(start 164.047 96.695)
+		(end 161.845 96.695)
 		(width 0.25)
 		(layer "F.Cu")
@@
 	)
 	(segment
-		(start 164.047 96.695)
-		(end 161.845 96.695)
+		(start 176.545 97.995)
+		(end 181.268187 93.271813)
+		(width 0.25)
+		(layer "F.Cu")
+		(net 17)
+	)
+	(segment
+		(start 188.367576 93.271813)
+		(end 193.72 93.271813)
 		(width 0.25)
 		(layer "F.Cu")
@@
 	)
 	(segment
+		(start 187.217344 93.271813)
+		(end 187.305344 93.183813)
+		(width 0.25)
+		(layer "F.Cu")
+		(net 17)
+	)
+	(segment
 		(start 181.268187 93.271813)
-		(end 193.72 93.271813)
+		(end 187.217344 93.271813)
 		(width 0.25)
 		(layer "F.Cu")
@@
 	)
 	(segment
+		(start 182.553187 95.811813)
+		(end 187.217344 95.811813)
+		(width 0.25)
+		(layer "F.Cu")
+		(net 28)
+	)
+	(segment
 		(start 176.545 101.82)
 		(end 176.545 102.995)
@@
 	)
 	(segment
+		(start 188.367576 95.811813)
+		(end 193.711813 95.811813)
+		(width 0.25)
+		(layer "F.Cu")
+		(net 28)
+	)
+	(segment
 		(start 164.295 99.245)
 		(end 162.845 97.795)
@@
 	)
 	(segment
-		(start 162.845 97.795)
-		(end 161.845 97.795)
+		(start 187.217344 95.811813)
+		(end 187.305344 95.723813)
 		(width 0.25)
 		(layer "F.Cu")
@@
 	)
 	(segment
+		(start 188.279576 95.723813)
+		(end 188.367576 95.811813)
+		(width 0.25)
+		(layer "F.Cu")
+		(net 28)
+	)
+	(segment
+		(start 162.845 97.795)
+		(end 161.845 97.795)
+		(width 0.25)
+		(layer "F.Cu")
+		(net 28)
+	)
+	(segment
 		(start 164.295 102.395)
 		(end 164.295 99.245)
@@
 	)
 	(segment
-		(start 182.553187 95.811813)
-		(end 193.711813 95.811813)
+		(start 187.305344 95.723813)
+		(end 188.279576 95.723813)
 		(width 0.25)
 		(layer "F.Cu")
@@
 	)
 	(segment
-		(start 213.72 122.32)
-		(end 215.22 122.32)
-		(width 0.2)
-		(layer "F.Cu")
-		(net 34)
-	)
-	(segment
 		(start 213.699813 122.299813)
 		(end 213.72 122.32)
@@
 		(net 34)
 	)
-	(via
-		(at 215.22 122.32)
-		(size 0.6)
-		(drill 0.3)
-		(layers "F.Cu" "B.Cu")
-		(net 34)
-	)
 	(segment
 		(start 231.72 127.09)
@@
 	(segment
 		(start 185.72 107.527353)
-		(end 185.72 90.32)
+		(end 185.72 96.32)
 		(width 0.25)
 		(layer "B.Cu")
@@
 	)
 	(segment
-		(start 185.72 90.32)
-		(end 181.72 86.32)
+		(start 185.72 96.32)
+		(end 181.72 92.32)
 		(width 0.25)
 		(layer "B.Cu")
@@
 	)
 	(segment
+		(start 181.72 92.32)
+		(end 181.72 86.32)
+		(width 0.25)
+		(layer "B.Cu")
+		(net 49)
+	)
+	(segment
 		(start 187.79246 96.899813)
 		(end 183.140187 96.899813)
@@
 	)
 	(segment
-		(start 181.72 103.82)
-		(end 182.22 103.82)
-		(width 0.2)
+		(start 174.6325 112.32)
+		(end 174.6325 110.9075)
+		(width 0.25)
 		(layer "F.Cu")
 		(net 51)
 	)
 	(segment
-		(start 184.060187 101.979813)
-		(end 187.79246 101.979813)
-		(width 0.2)
+		(start 174.6325 110.9075)
+		(end 181.72 103.82)
+		(width 0.25)
 		(layer "F.Cu")
 		(net 51)
 	)
 	(segment
-		(start 182.22 103.82)
-		(end 184.060187 101.979813)
+		(start 183.560187 101.979813)
+		(end 187.79246 101.979813)
 		(width 0.2)
 		(layer "F.Cu")
@@
 	)
 	(segment
-		(start 187.632647 101.82)
-		(end 187.79246 101.979813)
-		(width 0.25)
+		(start 181.72 103.82)
+		(end 183.560187 101.979813)
+		(width 0.2)
 		(layer "F.Cu")
 		(net 51)
 	)
 	(segment
-		(start 174.6325 112.32)
-		(end 174.6325 111.4075)
+		(start 187.632647 101.82)
+		(end 187.79246 101.979813)
 		(width 0.25)
 		(layer "F.Cu")
