File: E-throttle/E-throttle.kicad_pcb (KiCad board)
At the start: 2 copper layers, 100 x 100 mm, 68 parts, among them IC1 BTS441TG, J1 Conn_01x15_Socket, J2 Conn_01x15_Socket, J3 Conn_01x11, J4 Conn_01x11, J5 776087-1, J9 Micro_SD_Card, Q1 NMOS, SW1 SW_Push, U1 74HC123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

Commit message: changed 3V3 votlage regulator
Parts:
- U3: value LM317_SOT-223 -> TLV1117-33; footprint Package_TO_SOT_SMD:SOT-223-3_TabPin2 -> Package_TO_SOT_SMD:TO-252-3_TabPin2
- U4: value R-78E5.0-0.5 -> R-78E5.0-1.0
- moved U3 1.89 mm to (211.4, 72.4)
Routing:
- net /ESP_HEARTBEAT_L2: track 86.0 -> 76.6 mm, vias 1 -> 3
- net +3V3: track 310.8 -> 317.1 mm
- net +5V: track 109.8 -> 110.8 mm

Commit message: changed some resistor values
Parts:
- R11: value 392 -> 360
- R12, R9: value 240 -> 220
- R8: value 715 -> 665
Routing:
- net /CAN-L: vias 3 -> 1
Changed lines of the file:
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@@
 			)
 		)
-		(property "Value" "715"
+		(property "Value" "665"
 			(at 0.0875 1.5 0)
 			(layer "F.Fab")
@@
 		(sheetname "/")
 		(sheetfile "E-throttle.kicad_sch")
-		(attr smd dnp)
+		(attr smd)
 		(fp_line
 			(start -2.06 -2.56)
@@
 			)
 		)
-		(property "Value" "392"
+		(property "Value" "360"
 			(at 0 1.65 180)
 			(layer "F.Fab")
@@
 			)
 		)
-		(property "Value" "240"
+		(property "Value" "220"
 			(at 0 1.65 0)
 			(layer "F.Fab")
@@
 			)
 		)
-		(property "Value" "240"
+		(property "Value" "220"
 			(at 0 1.65 0)
 			(layer "F.Fab")
@@
 	)
 	(segment
-		(start 238.45 123.59)
-		(end 236.72 125.32)
-		(width 0.2)
-		(layer "F.Cu")
-		(net 41)
-	)
-	(segment
-		(start 238.45 121.32)
-		(end 238.45 123.59)
-		(width 0.2)
-		(layer "F.Cu")
-		(net 41)
-	)
-	(segment
 		(start 233.68 128.36)
 		(end 233.72 128.32)
@@
 	)
 	(via
-		(at 238.45 121.32)
-		(size 0.6)
-		(drill 0.3)
-		(layers "F.Cu" "B.Cu")
-		(net 41)
-	)
-	(via
 		(at 233.72 128.32)
 		(size 0.6)
@@
 		(net 41)
 	)
-	(via
-		(at 236.72 125.32)
-		(size 0.6)
-		(drill 0.3)
-		(layers "F.Cu" "B.Cu")
-		(net 41)
-	)
 	(segment
-		(start 238.45 75.332843)
-		(end 231.22 68.102843)
+		(start 238.45 123.59)
+		(end 233.72 128.32)
 		(width 0.2)
 		(layer "B.Cu")
@@
 	)
 	(segment
-		(start 233.72 128.32)
-		(end 236.72 125.32)
+		(start 221.783414 37.8075)
+		(end 231.22 47.244085)
 		(width 0.2)
 		(layer "B.Cu")
@@
 	)
 	(segment
-		(start 221.783414 37.8075)
-		(end 203.7325 37.8075)
+		(start 238.45 75.332843)
+		(end 238.45 123.59)
 		(width 0.2)
 		(layer "B.Cu")
@@
 	)
 	(segment
-		(start 238.45 121.32)
-		(end 238.45 75.332843)
+		(start 203.7325 37.8075)
+		(end 221.783414 37.8075)
 		(width 0.2)
 		(layer "B.Cu")
@@
 	(segment
 		(start 231.22 47.244085)
-		(end 221.783414 37.8075)
+		(end 231.22 68.102843)
 		(width 0.2)
 		(layer "B.Cu")
@@
 	)
 	(segment
-		(start 231.22 68.102843)
-		(end 231.22 47.244085)
+		(start 201.72 39.82)
+		(end 203.7325 37.8075)
 		(width 0.2)
 		(layer "B.Cu")
@@
 	)
 	(segment
-		(start 203.7325 37.8075)
-		(end 201.72 39.82)
+		(start 231.22 68.102843)
+		(end 238.45 75.332843)
 		(width 0.2)
 		(layer "B.Cu")
